File: new_file.kicad_pcb (KiCad board)
At the start: 2 copper layers, 35 x 25 mm, 12 parts, among them J1 SWD, J2 VDD, J3 I2C, U1 MDBT42Q-512K, U2 SHT4x

Commit message: Add files via upload
Parts:
- C1: footprint bt_holder:cap_100nf -> bt_holder:cap_100nf (2)
- moved R2 2.50 mm to (176.5, 77.0), turned to -90 degrees
- moved C1 1.12 mm to (181.0, 81.0)
Routing:
- net GND: track 56.3 -> 37.1 mm, vias 5 -> 10
- net /VDD: track 23.2 -> 4.09 mm, vias 3 -> 0
- net /SDA: track 26.8 -> 17.0 mm, vias 0 -> 2
- net /CLK: track 12.3 -> 10.4 mm, vias 0 -> 2
- net /RST: track 16.6 -> 18.4 mm, vias 0 -> 2
- net /SCL: track 24.8 -> 22.9 mm, vias 0 -> 2
